File: POWER.kicad_sch (KiCad schematic)
At the start: 59 parts, among them CN3 1.25mm-2P socket, CN4 1.25mm-2P socket, Q1 AO3401A, U1 USBLC6-2P6, U2 TPS63900, U3 CH340E, U4 TPS22917DBV, U5 TPS22917DBV, U6 BQ25185DLHR

Commit message: prod files
Parts:
- C10, C9: LCSC (none) -> C76971
- C3, C5: LCSC (none) -> C1525
- C4, C49: LCSC (none) -> C45783
- C50, C6, C7: LCSC (none) -> C15525
- C51, C52: LCSC (none) -> C52923
- CN3, CN4: LCSC (none) -> C43462
- D1, D2, D5: LCSC (none) -> C191023
- D3, D6, D7, D8, D9: LCSC (none) -> C22355736
- D4: LCSC (none) -> C52148463
- L1: LCSC (none) -> C3151182
- Q1: LCSC (none) -> C15127
- R1: LCSC (none) -> C26083
- R10, R5: LCSC (none) -> C17168
- R11, R12, R7: LCSC (none) -> C11702
- R14, R15: LCSC (none) -> C25741
- R16, R19, R8: LCSC (none) -> C25744
- R17, R18, R20: LCSC (none) -> C25900
- R4: LCSC (none) -> C27176
- R6: LCSC (none) -> C25887
- R9: LCSC (none) -> C4961
- U2: LCSC (none) -> C1518762
- U3: LCSC (none) -> C99652
- U4, U5: LCSC (none) -> C2681320
- U6: LCSC (none) -> C19725033
