File: RF.kicad_sch (KiCad schematic)
At the start: 20 parts, among them J2 Conn_Coaxial_Small, J3 Conn_Coaxial_Small, U10 RFANT3216120A5T, U9 SKY65943-11

Commit message: prod files
Parts:
- C36, C39: LCSC (none) -> C1525
- C38: LCSC (none) -> C76917
- J2, J3: LCSC (none) -> C22418213
- L10: LCSC (none) -> C88970
- L8: LCSC (none) -> C108965
- L9: LCSC (none) -> C113122
- R36: LCSC (none) -> C11702
- R37, R38: LCSC (none) -> C17168
- U10: LCSC (none) -> C127629
- U9: LCSC (none) -> C2654442
