File: SIM.kicad_sch (KiCad schematic)
At the start: 4 parts, among them IC1 SIM-S-IO3-MFF2-2-LP, J4 JAE_SIM_Card_SF72S006

Commit message: prod files
Parts:
- C47: LCSC (none) -> C15195
- J4: LCSC (none) -> C2977286
- L11: LCSC (none) -> C2869050
Changed lines of the file:
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@@
 	(title_block
 		(title "MIRA")
-		(date "2026-10-23")
+		(date "2026-10-25")
 		(rev "1.0")
 		(company "Pierluigi Colangeli")
@@
 		(effects
 			(font
-				(face "Avenir Black")
+				(face "KiCad Font")
 				(size 2.54 2.54)
 				(thickness 0.508)
@@
 			)
 		)
+		(property "JLCPCB Part #" ""
+			(at 43.18 90.17 0)
+			(hide yes)
+			(show_name no)
+			(do_not_autoplace no)
+			(effects
+				(font
+					(size 1.27 1.27)
+				)
+			)
+		)
 		(pin "5"
 		)
@@
 			)
 		)
+		(property "LCSC" "C15195"
+			(at 109.22 30.4862 0)
+			(hide yes)
+			(show_name no)
+			(do_not_autoplace no)
+			(effects
+				(font
+					(size 1.27 1.27)
+				)
+			)
+		)
+		(property "JLCPCB Part #" ""
+			(at 106.68 31.75 0)
+			(hide yes)
+			(show_name no)
+			(do_not_autoplace no)
+			(effects
+				(font
+					(size 1.27 1.27)
+				)
+			)
+		)
 		(pin "1"
 		)
@@
 			)
 		)
+		(property "LCSC" "C2977286"
+			(at 125.984 36.322 0)
+			(hide yes)
+			(show_name no)
+			(do_not_autoplace no)
+			(effects
+				(font
+					(size 1.27 1.27)
+				)
+			)
+		)
+		(property "JLCPCB Part #" ""
+			(at 121.92 53.34 0)
+			(hide yes)
+			(show_name no)
+			(do_not_autoplace no)
+			(effects
+				(font
+					(size 1.27 1.27)
+				)
+			)
+		)
 		(pin "C5"
 		)
@@
 				)
 			)
+		)
+		(property "LCSC" "C2869050"
+			(at 82.55 41.656 0)
+			(hide yes)
+			(show_name no)
+			(do_not_autoplace no)
+			(effects
+				(font
+					(size 1.27 1.27)
+				)
+			)
+		)
+		(property "JLCPCB Part #" ""
+			(at 82.55 50.8 0)
+			(hide yes)
+			(show_name no)
+			(do_not_autoplace no)
+			(effects
+				(font
+					(size 1.27 1.27)
+				)
+			)
