File: nRF54L.kicad_sch (KiCad schematic)
At the start: 38 parts, among them CN1 FTSH-105, U16 APHF1608LSEEQBDZGKC, U7 nRF54L15-QFXX, X1 32MHz, X2 32.768KHz

Commit message: more codes lcsc
Parts:
- L4, L5: LCSC (none) -> C206424
Changed lines of the file:
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@@
+			)
+		)
+		(property "LCSC" "C206424"
+			(at 190.5 100.33 90)
+			(hide yes)
+			(show_name no)
+			(do_not_autoplace no)
+			(effects
+				(font
+					(size 1.27 1.27)
+				)
 			)
 		)
@@
 				)
 			)
+		)
+		(property "LCSC" "C206424"
+			(at 203.2 100.33 90)
+			(hide yes)
+			(show_name no)
+			(do_not_autoplace no)
+			(effects
+				(font
+					(size 1.27 1.27)
+				)
+			)

Commit message: prod files
Parts:
- C12: LCSC (none) -> C15525
- C13, C14, C16, C19, C48: LCSC (none) -> C49062
- C15: LCSC (none) -> C76917
- C17: LCSC (none) -> C76926
- C18, C22: LCSC (none) -> C318539
- C20: LCSC (none) -> C88913
- C21: LCSC (none) -> C161374
- C25: LCSC (none) -> C76901
- CN1: LCSC (none) -> C448647
- FB1: LCSC (none) -> C97850
- L6: LCSC (none) -> C85670
- R21: LCSC (none) -> C11702
- R22: LCSC (none) -> C25121
- R23, R24, R25, R26, R27: LCSC (none) -> C25900
- R28: LCSC (none) -> C17168
- R41: LCSC (none) -> C26083
- R42: LCSC (none) -> C25778
- U16: LCSC (none) -> C3019171
- U7: LCSC (none) -> C42458750
- X1: LCSC (none) -> C655046
- X2: LCSC (none) -> C596929
