File: nRF9151.kicad_sch (KiCad schematic)
At the start: 25 parts, among them CN2 FTSH-105, Q2 DMN2990UFA-7B, Q3 DMP22D4UFA-7B, Q4 DMN2990UFA-7B, U8 nRF9151-LAXX

Commit message: prod files
Parts:
- C27: LCSC (none) -> C1548
- C28, C32, C34: LCSC (none) -> C1525
- C29: LCSC (none) -> C16780
- C30: LCSC (none) -> C15525
- C31, C33: LCSC (none) -> C19666
- CN2: LCSC (none) -> C448647
- L7: LCSC (none) -> C88970
- Q2, Q4: LCSC (none) -> C151598
- Q3: LCSC (none) -> C2983692
- R29, R31, R34: LCSC (none) -> C26083
- R30, R32, R33: LCSC (none) -> C25741
- R35: LCSC (none) -> C11702
- U8: LCSC (none) -> C22397843
